Commit message: change joint translations to sync with mesh rotations

File: popi_software/popi/popi_description/xacro/popi_champ.xacro (robot description, xacro)
@@ -181,5 +181,5 @@
 	    <inertial>
 	      	<origin xyz="-0.11389 -0.00555 0.00901"
-	        		rpy="0 -1.5708 0" />
+	        		rpy="0 -1.495 0" />
 	      	<mass value="${masse_hjambe}" />
 	      	<inertia 	ixx="0.01032" 	ixy="-0.00226" 	ixz="0.01011"
@@ -189,5 +189,5 @@
 	    <visual>
 	     	<origin xyz="0 0 0"
-	        		rpy="0 -1.5708 0" />
+	        		rpy="0 -1.495 0" />
 	      	<geometry>
 	        	<mesh filename="package://popi_description/meshes/HJambeAVG.STL" />
@@ -387,5 +387,5 @@
 	    <inertial>
 	      	<origin xyz="-0.11389 -0.00555 0.00901"
-	        		rpy="0 -1.5708 0" />
+	        		rpy="0 -1.495 0" />
 	      	<mass value="${masse_hjambe}" />
 	      	<inertia 	ixx="0.01032" 	ixy="-0.00226"	ixz="0.01011"
@@ -395,5 +395,5 @@
 	    <visual>
 	      	<origin xyz="0 0 0"
-	        		rpy="0 -1.5708 0" />
+	        		rpy="0 -1.495 0" />
 	     	<geometry>
 	        	<mesh filename="package://popi_description/meshes/HJambeARG.STL" />
@@ -489,5 +489,5 @@
   	</joint>
   	<joint name="coudeAVD" type="revolute">
-	    <origin xyz="-0.35192 0 -0.041509"
+	    <origin xyz="0.041509 0 -0.35192"
 	      		rpy="0 0 0" />
 	    <parent link="HJambeAVD" />
@@ -502,5 +502,5 @@
   	</joint>
   	<joint name="piedAVD" type="fixed">
-	    <origin xyz="0.29604 0 -0.015"
+	    <origin xyz="-0.015 0 -0.29604"
 	      		rpy="0 0 0" />
 	    <parent link="BJambeAVD" />
@@ -538,5 +538,5 @@
   	</joint>
   	<joint name="coudeAVG" type="revolute">
-	    <origin xyz="-0.35192 0 -0.041509"
+	    <origin xyz="0.041509 0 -0.35192"
 	      		rpy="0 0 0" />
 	    <parent link="HJambeAVG" />
@@ -551,5 +551,5 @@
   	</joint>
   	<joint name="piedAVG" type="fixed">
-    	<origin xyz="0.29604 0 -0.015"
+    	<origin xyz="-0.015 0 -0.29604"
       			rpy="0 0 0" />
 	    <parent link="BJambeAVG" />
@@ -587,5 +587,5 @@
 	</joint>
 	<joint name="coudeARD" type="revolute">
-	    <origin xyz="-0.35192 0 -0.041509"
+	    <origin xyz="0.041509 0 -0.35192"
 	      		rpy="0 0 0" />
 	    <parent link="HJambeARD" />
@@ -600,5 +600,5 @@
 	</joint>
 	<joint name="piedARD" type="fixed">
-	    <origin xyz="0.29604 0 -0.015"
+	    <origin xyz="-0.015 0 -0.29604"
 	      		rpy="0 0 0" />
 	    <parent link="BJambeARD" />
@@ -636,5 +636,5 @@
   	</joint>
 	<joint name="coudeARG" type="revolute">
-		<origin xyz="-0.35192 0 -0.041509"
+		<origin xyz="0.041509 0 -0.35192"
 		  		rpy="0 0 0" />
 		<parent link="HJambeARG" />
@@ -649,5 +649,5 @@
 	</joint>
 	<joint name="piedARG" type="fixed">
-	    <origin xyz="0.29604 0 -0.015"
+	    <origin xyz="-0.015 0 -0.29604"
 	      		rpy="0 0 0" />
 	    <parent link="BJambeARG" />

Commit message: change joint limits to sync with joint rotational changes

File: popi_software/popi/popi_description/xacro/popi_champ.xacro (robot description, xacro)
@@ -481,6 +481,6 @@
 	    <child  link="HJambeAVD" />
 	    <axis   xyz="0 -1 0" />
-	    <limit  lower="${lower_epaule}"
-      			upper="${upper_epaule}"
+	    <limit  lower="-1.5708"
+      			upper="1.5708"
       			effort="${effort_epaule}"
       			velocity="${vel_epaule}" />
@@ -494,6 +494,6 @@
 	    <child  link="BJambeAVD" />
 	    <axis   xyz="0 1 0" />
-	    <limit  lower="${lower_coude}"
-      			upper="${upper_coude}"
+	    <limit  lower="-0.26"
+      			upper="1.92"
       			effort="${effort_coude}"
       			velocity="${vel_coude}" />
@@ -530,6 +530,6 @@
 	    <child  link="HJambeAVG" />
 	    <axis   xyz="0 -1 0" />
-	    <limit  lower="${lower_epaule}"
-      			upper="${upper_epaule}"
+	    <limit  lower="-1.5708"
+      			upper="1.5708"
       			effort="${effort_epaule}"
       			velocity="${vel_epaule}" />
@@ -543,6 +543,6 @@
 	    <child  link="BJambeAVG" />
 	    <axis   xyz="0 1 0" />
-	    <limit  lower="${lower_coude}"
-      			upper="${upper_coude}"
+	    <limit  lower="-0.26"
+      			upper="1.92"
       			effort="${effort_coude}"
       			velocity="${vel_coude}" />
@@ -579,6 +579,6 @@
 	    <child  link="HJambeARD" />
 	    <axis   xyz="0 -1 0" />
-	    <limit  lower="${lower_epaule}"
-      			upper="${upper_epaule}"
+	    <limit  lower="-1.5708"
+      			upper="1.5708"
       			effort="${effort_epaule}"
       			velocity="${vel_epaule}" />
@@ -592,6 +592,6 @@
 	    <child  link="BJambeARD" />
 	    <axis   xyz="0 1 0" />
-	    <limit  lower="${lower_coude}"
-      			upper="${upper_coude}"
+	    <limit  lower="-0.26"
+      			upper="1.92"
       			effort="${effort_coude}"
       			velocity="${vel_coude}" />
@@ -628,6 +628,6 @@
 	    <child  link="HJambeARG" />
 	    <axis   xyz="0 -1 0" />
-	    <limit  lower="${lower_epaule}"
-      			upper="${upper_epaule}"
+	    <limit  lower="-1.5708"
+      			upper="1.5708"
       			effort="${effort_epaule}"
       			velocity="${vel_epaule}" />
@@ -641,6 +641,6 @@
 		<child  link="BJambeARG" />
 		<axis   xyz="0 1 0" />
-		<limit  lower="${lower_coude}"
-      			upper="${upper_coude}"
+		<limit  lower="-0.26"
+      			upper="1.92"
       			effort="${effort_coude}"
       			velocity="${vel_coude}" />

Commit message: discretized collisions by using geometrical shapes

File: popi_software/popi/popi_description/xacro/popi_champ.xacro (robot description, xacro)
@@ -40,8 +40,8 @@
 	    </visual>
 	    <collision>
-	      	<origin xyz="0 0 0"
+	      	<origin xyz="0 0 -0.035"
 	        	  	rpy="0 0 0" />
 	      	<geometry>
-	        	<mesh filename="package://popi_description/meshes/Bati.STL" />
+          		<box size="0.84 0.4 0.2" />
 	      	</geometry>
 	    </collision>
@@ -68,8 +68,8 @@
     	</visual>
     	<collision>
-      		<origin xyz="0 0 0"
-        			rpy="0 0 0" />
-      		<geometry>
-        		<mesh filename="package://popi_description/meshes/EpauleAVD.STL" />
+      		<origin xyz="0 0.075 0"
+        			rpy="0 0 0" />
+      		<geometry>
+          		<box size="0.15 0.15 0.12" />
       		</geometry>
     	</collision>
@@ -77,6 +77,6 @@
   	<link name="HJambeAVD">
     	<inertial>
-     		<origin xyz="-0.11331 0.00512 0.01743"
-        			rpy="0 -1.5708 0" />
+     		<origin xyz="0.01743 0.00512 -0.11331"
+        			rpy="0 0 0" />
       		<mass value="${masse_hjambe}" />
       		<inertia 	ixx="0.00899" 	ixy="0.00215" 	ixz="0.00647"
@@ -93,8 +93,8 @@
     	</visual>
     	<collision>
-      		<origin xyz="0 0 0"
-        			rpy="0 0 0" />
-      		<geometry>
-        		<mesh filename="package://popi_description/meshes/HJambeAVD.STL" />
+      		<origin xyz="0 0 -0.15"
+        			rpy="0 0 0" />
+      		<geometry>
+          		<box size="0.1 0.1 -0.43" />
       		</geometry>
     	</collision>
@@ -102,6 +102,6 @@
   	<link name="BJambeAVD">
     	<inertial>
-      		<origin xyz="0.11761 0 -0.012387"
-        			rpy="0 1.5708 0" />
+      		<origin xyz="-0.012387 0 -0.11761"
+        			rpy="0 0 0" />
       		<mass value="${masse_bjambe}" />
       		<inertia 	ixx="0.000103" 	ixy="0.000000" 	ixz="-0.00019"
@@ -118,8 +118,8 @@
     	</visual>
     	<collision>
-      		<origin xyz="0 0 0"
-        			rpy="0 0 0" />
-      		<geometry>
-        		<mesh filename="package://popi_description/meshes/BJambeAVD.STL" />
+      		<origin xyz="0 0 -0.08"
+        			rpy="0 0 0" />
+      		<geometry>
+          		<box size="0.05 0.05 -0.32" />
       		</geometry>
     	</collision>
@@ -143,8 +143,8 @@
     	</visual>
     	<collision>
-      		<origin xyz="0 0 0"
+      		<origin xyz="0 0 0.033"
         	  		rpy="0 0 0" />
       		<geometry>
-        		<mesh filename="package://popi_description/meshes/PiedAVD.STL" />
+        		<sphere radius="0.0335" />
       		</geometry>
     	</collision>
@@ -171,8 +171,8 @@
     	</visual>
     	<collision>
-      		<origin xyz="0 0 0"
-        			rpy="0 0 0" />
-      		<geometry>
-        		<mesh filename="package://popi_description/meshes/EpauleAVG.STL" />
+      		<origin xyz="0 -0.075 0"
+        			rpy="0 0 0" />
+      		<geometry>
+          		<box size="0.15 0.15 0.12" />
       		</geometry>
     	</collision>
@@ -180,5 +180,5 @@
 	<link name="HJambeAVG">
 	    <inertial>
-	      	<origin xyz="-0.11389 -0.00555 0.00901"
+	      	<origin xyz="0.00901 -0.00555 -0.11389"
 	        		rpy="0 -1.495 0" />
 	      	<mass value="${masse_hjambe}" />
@@ -195,16 +195,16 @@
 	      	<material name="darkgrey"/>
 	    </visual>
-	    <collision>
-	      	<origin xyz="0 0 0"
-	        		rpy="0 0 0" />
-	      		<geometry>
-	        		<mesh filename="package://popi_description/meshes/HJambeAVG.STL" />
-	      		</geometry>
-	    </collision>
+    	<collision>
+      		<origin xyz="0 0 -0.15"
+        			rpy="0 0 0" />
+      		<geometry>
+          		<box size="0.1 0.1 -0.43" />
+      		</geometry>
+    	</collision>
 	</link>
 	<link name="BJambeAVG">
 	    <inertial>
-	      	<origin xyz="0.11761 0 -0.012387"
-	        		rpy="0 1.5708 0" />
+	      	<origin xyz="-0.012387 0 -0.11761"
+	        		rpy="0 0 0" />
 	      	<mass value="${masse_bjambe}" />
 	      	<inertia 	ixx="0.000103" 	ixy="0.000000" 	ixz="-0.00019"
@@ -220,11 +220,11 @@
 	      	<material name="white"/>
 	    </visual>
-	    <collision>
-	      	<origin xyz="0 0 0"
-        		  	rpy="0 0 0" />
-	      	<geometry>
-	        	<mesh filename="package://popi_description/meshes/BJambeAVG.STL" />
-	      	</geometry>
-	    </collision>
+    	<collision>
+      		<origin xyz="0 0 -0.08"
+        			rpy="0 0 0" />
+      		<geometry>
+          		<box size="0.05 0.05 -0.32" />
+      		</geometry>
+    	</collision>
 	</link>
 	<link name="PiedAVG">
@@ -246,9 +246,9 @@
 	    </visual>
 	    <collision>
-	      	<origin xyz="0 0 0"
-	        	  	rpy="0 0 0" />
-	      	<geometry>
-	        	<mesh filename="package://popi_description/meshes/PiedAVG.STL" />
-	      	</geometry>
+      		<origin xyz="0 0 0.033"
+        	  		rpy="0 0 0" />
+      		<geometry>
+        		<sphere radius="0.0335" />
+      		</geometry>
     	</collision>
   	</link>
@@ -274,8 +274,8 @@
 	    </visual>
 	    <collision>
-	      	<origin xyz="0 0 0"
+	      	<origin xyz="0 0.075 0"
 	        		rpy="0 0 0" />
 	        <geometry>
-	        	<mesh filename="package://popi_description/meshes/EpauleARD.STL" />
+          		<box size="0.15 0.15 0.12" />
 	      	</geometry>
 	    </collision>
@@ -283,6 +283,6 @@
 	<link name="HJambeARD">
 	    <inertial>
-	     	<origin xyz="-0.11331 0.00512 0.01743"
-	        		rpy="0 -1.5708 0" />
+	     	<origin xyz="0.01743 0.00512 -0.11331"
+	        		rpy="0 0 0" />
 	      	<mass value="${masse_hjambe}" />
 	      	<inertia 	ixx="0.00899" 	ixy="0.00215" 	ixz="0.00647"
@@ -298,16 +298,16 @@
 	      	<material name="darkgrey"/>
 	    </visual>
-	    <collision>
-	      	<origin xyz="0 0 0"
-	        		rpy="0 0 0" />
-	      	<geometry>
-	        	<mesh filename="package://popi_description/meshes/HJambeARD.STL" />
-	      	</geometry>
-	    </collision>
+    	<collision>
+      		<origin xyz="0 0 -0.15"
+        			rpy="0 0 0" />
+      		<geometry>
+          		<box size="0.1 0.1 -0.43" />
+      		</geometry>
+    	</collision>
 	</link>
   	<link name="BJambeARD">
 	    <inertial>
-	      	<origin xyz="0.11761 0 -0.012387"
-	        		rpy="0 1.5708 0" />
+	      	<origin xyz="-0.012387 0 -0.11761"
+	        		rpy="0 0 0" />
 	      	<mass value="${masse_bjambe}" />
 	      	<inertia 	ixx="0.000103" 	ixy="0.000000" 	ixz="-0.00019"
@@ -324,10 +324,10 @@
 	    </visual>
 	    <collision>
-	      	<origin xyz="0 0 0"
-	        		rpy="0 0 0" />
-	      	<geometry>
-	        	<mesh filename="package://popi_description/meshes/BJambeARD.STL" />
-	      	</geometry>
-	    </collision>
+      		<origin xyz="0 0 -0.08"
+        			rpy="0 0 0" />
+      		<geometry>
+          		<box size="0.05 0.05 -0.32" />
+      		</geometry>
+    	</collision>
   	</link>
 	<link name="PiedARD">
@@ -349,10 +349,10 @@
 	    </visual>
 	    <collision>
-	      	<origin xyz="0 0 0"
-	        		rpy="0 0 0" />
-	      	<geometry>
-	        	<mesh filename="package://popi_description/meshes/PiedARD.STL" />
-	      	</geometry>
-	    </collision>
+      		<origin xyz="0 0 0.033"
+        	  		rpy="0 0 0" />
+      		<geometry>
+        		<sphere radius="0.0335" />
+      		</geometry>
+    	</collision>
 	</link>
 <!--**************************************************************************************-->
@@ -377,8 +377,8 @@
     	</visual>
     	<collision>
-      		<origin xyz="0 0 0"
-        			rpy="0 0 0" />
-      		<geometry>
-        		<mesh filename="package://popi_description/meshes/EpauleARG.STL" />
+      		<origin xyz="0 -0.075 0"
+        			rpy="0 0 0" />
+      		<geometry>
+          		<box size="0.15 0.15 0.12" />
       		</geometry>
     	</collision>
@@ -386,5 +386,5 @@
 	<link name="HJambeARG">
 	    <inertial>
-	      	<origin xyz="-0.11389 -0.00555 0.00901"
+	      	<origin xyz="0.00901 -0.00555 -0.11389"
 	        		rpy="0 -1.495 0" />
 	      	<mass value="${masse_hjambe}" />
@@ -401,16 +401,16 @@
 	      	<material name="darkgrey"/>
 	    </visual>
-	    <collision>
-	      	<origin xyz="0 0 0"
-	        		rpy="0 0 0" />
-	     	<geometry>
-	        	<mesh filename="package://popi_description/meshes/HJambeARG.STL" />
-	      	</geometry>
-	    </collision>
+    	<collision>
+      		<origin xyz="0 0 -0.15"
+        			rpy="0 0 0" />
+      		<geometry>
+          		<box size="0.1 0.1 -0.43" />
+      		</geometry>
+    	</collision>
 	</link>
 	<link name="BJambeARG">
 	    <inertial>
-	      	<origin xyz="0.11761 0.0 -0.012387"
-	        		rpy="0 1.5708 0" />
+	      	<origin xyz="-0.012387 0 -0.11761"
+	        		rpy="0 0 0" />
 	      	<mass value="${masse_bjambe}" />
 	      	<inertia ixx="0.000103" 	ixy="0.000000" 	ixz="-0.00019"
@@ -427,10 +427,10 @@
 	    </visual>
 	    <collision>
-	      	<origin xyz="0 0 0"
-	        		rpy="0 0 0" />
-	      	<geometry>
-	        	<mesh filename="package://popi_description/meshes/BJambeARG.STL" />
-	      	</geometry>
-	    </collision>
+      		<origin xyz="0 0 -0.08"
+        			rpy="0 0 0" />
+      		<geometry>
+          		<box size="0.05 0.05 -0.32" />
+      		</geometry>
+    	</collision>
 	</link>
 	<link name="PiedARG">
@@ -452,10 +452,10 @@
 	    </visual>
 	    <collision>
-	      	<origin xyz="0 0 0"
-	        		rpy="0 0 0" />
-	      	<geometry>
-	        	<mesh filename="package://popi_description/meshes/PiedARG.STL" />
-	      	</geometry>
-	    </collision>
+      		<origin xyz="0 0 0.033"
+        	  		rpy="0 0 0" />
+      		<geometry>
+        		<sphere radius="0.0335" />
+      		</geometry>
+    	</collision>
 	</link>
 <!--**************************************************************************************-->
@@ -467,5 +467,5 @@
     	<parent link="Bati" />
     	<child  link="EpauleAVD" />
-    	<axis   xyz="-1 0 0" />
+    	<axis   xyz="1 0 0" />
     	<limit  lower="${lower_aile}"
       			upper="${upper_aile}"
@@ -480,5 +480,5 @@
 	    <parent link="EpauleAVD" />
 	    <child  link="HJambeAVD" />
-	    <axis   xyz="0 -1 0" />
+	    <axis   xyz="0 1 0" />
 	    <limit  lower="-1.5708"
       			upper="1.5708"
@@ -529,5 +529,5 @@
 	    <parent link="EpauleAVG" />
 	    <child  link="HJambeAVG" />
-	    <axis   xyz="0 -1 0" />
+	    <axis   xyz="0 1 0" />
 	    <limit  lower="-1.5708"
       			upper="1.5708"
@@ -565,5 +565,5 @@
 	    <parent link="Bati" />
 	    <child  link="EpauleARD" />
-	    <axis   xyz="-1 0 0" />
+	    <axis   xyz="1 0 0" />
 	    <limit  lower="${lower_aile}"
       			upper="${upper_aile}"
@@ -578,5 +578,5 @@
 	    <parent link="EpauleARD" />
 	    <child  link="HJambeARD" />
-	    <axis   xyz="0 -1 0" />
+	    <axis   xyz="0 1 0" />
 	    <limit  lower="-1.5708"
       			upper="1.5708"
@@ -627,5 +627,5 @@
 	    <parent link="EpauleARG" />
 	    <child  link="HJambeARG" />
-	    <axis   xyz="0 -1 0" />
+	    <axis   xyz="0 1 0" />
 	    <limit  lower="-1.5708"
       			upper="1.5708"
